File: kicad/PSP-603_USB.kicad_pcb (KiCad board)
At the start: 2 copper layers, 33 parts, among them J1 10118194-0001LF, J2 826947-4, U1 93LC56BT-I/OT, U2 FT232HL-Reel, X1 ABM10AIG-12.000MHZ-4Z-T3

Commit message: Signed-off-by: Chris Stook <chris@chrisstook.com>
Parts:
- added C14: C1005X7R1H104K050BB, Standard_Footprints:C0402, F.Cu at (159.4, 52.7)
- added U3: SN74LV1T34DBVR, Standard_Footprints:TSOT-23-5, F.Cu at (159.4, 55.2)
Connections:
- U2 pad 13: /UART_TX -> Net-(U2-Pad13)
Changed lines of the file:
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@@
 (kicad_pcb (version 4) (host pcbnew 4.0.1-stable)
   (general
-    (links 91)
-    (no_connects 89)
+    (links 96)
+    (no_connects 94)
     (area 0 0 0 0)
     (thickness 1.6)
@@
     (tracks 0)
     (zones 0)
-    (modules 33)
-    (nets 42)
+    (modules 35)
+    (nets 44)
   )
   (page A4)
@@
     (pad_to_mask_clearance 0.2)
     (aux_axis_origin 0 0)
-    (visible_elements FFFCF77F)
+    (visible_elements 7FFEFFFF)
     (pcbplotparams
       (layerselection 0x00030_80000001)
@@
   (net 40 "Net-(U2-Pad29)")
   (net 41 "Net-(U2-Pad33)")
+  (net 42 "Net-(U2-Pad13)")
+  (net 43 "Net-(U3-Pad1)")
   (net_class Default "This is the default net class."
     (clearance 0.2032)
@@
     (add_net "Net-(R5-Pad2)")
     (add_net "Net-(R7-Pad2)")
+    (add_net "Net-(U2-Pad13)")
     (add_net "Net-(U2-Pad15)")
     (add_net "Net-(U2-Pad16)")
@@
     (add_net "Net-(U2-Pad29)")
     (add_net "Net-(U2-Pad33)")
+    (add_net "Net-(U3-Pad1)")
   )
   (module Standard_Footprints:C0603 (layer F.Cu)
@@
       (net 7 /VCCD))
     (pad 13 smd oval (at -2.75 4.2 180) (size 0.25 1.5) (layers F.Cu F.Paste F.Mask)
-      (net 27 /UART_TX))
+      (net 42 "Net-(U2-Pad13)"))
     (pad 14 smd oval (at -2.25 4.2 180) (size 0.25 1.5) (layers F.Cu F.Paste F.Mask)
       (net 28 /UART_RX))
@@
       (net 1 GND))
   )
+  (module Standard_Footprints:TSOT-23-5 (layer F.Cu)
+    (at 159.385 55.245)
+    (fp_text reference U3 (at 0 2.77) (layer F.SilkS)
+      (effects (font (size 1.2 1.2) (thickness 0.2)))
+    )
+    (fp_text value SN74LV1T34DBVR (at 0 -2.77) (layer F.SilkS)
+      (effects (font (size 1.2 1.2) (thickness 0.2)))
+    )
+    (fp_line (start 0.62 -1.57) (end -0.38 -0.57) (layer F.SilkS) (width 0.2))
+    (fp_line (start -0.38 -0.57) (end -0.38 1.57) (layer F.SilkS) (width 0.2))
+    (fp_line (start -0.38 1.57) (end 0.38 1.57) (layer F.SilkS) (width 0.2))
+    (fp_line (start 0.38 1.57) (end 0.38 -1.57) (layer F.SilkS) (width 0.2))
+    (fp_line (start 0.38 -1.57) (end 0.62 -1.57) (layer F.SilkS) (width 0.2))
+    (pad 1 smd rect (at -1.3 -0.95) (size 1.22 0.62) (layers F.Cu F.Paste F.Mask)
+      (net 43 "Net-(U3-Pad1)"))
+    (pad 2 smd rect (at -1.3 0) (size 1.22 0.62) (layers F.Cu F.Paste F.Mask)
+      (net 42 "Net-(U2-Pad13)"))
+    (pad 3 smd rect (at -1.3 0.95) (size 1.22 0.62) (layers F.Cu F.Paste F.Mask)
+      (net 1 GND))
+    (pad 5 smd rect (at 1.3 -0.95) (size 1.22 0.62) (layers F.Cu F.Paste F.Mask)
+      (net 3 /VBUS))
+    (pad 4 smd rect (at 1.3 0.95) (size 1.22 0.62) (layers F.Cu F.Paste F.Mask)
+      (net 27 /UART_TX))
+  )
+  (module Standard_Footprints:C0402 (layer F.Cu)
+    (at 159.385 52.705)
+    (descr "Capacitor SMD 0402, reflow soldering, AVX (see smccp.pdf)")
+    (tags "capacitor 0402")
+    (attr smd)
+    (fp_text reference C14 (at 0 -1.7) (layer F.SilkS)
+      (effects (font (size 1 1) (thickness 0.15)))
+    )
+    (fp_text value C1005X7R1H104K050BB (at 0 1.7) (layer F.SilkS)
+      (effects (font (size 1 1) (thickness 0.15)))
+    )
+    (fp_line (start -1.15 -0.6) (end 1.15 -0.6) (layer F.CrtYd) (width 0.05))
+    (fp_line (start -1.15 0.6) (end 1.15 0.6) (layer F.CrtYd) (width 0.05))
+    (fp_line (start -1.15 -0.6) (end -1.15 0.6) (layer F.CrtYd) (width 0.05))
+    (fp_line (start 1.15 -0.6) (end 1.15 0.6) (layer F.CrtYd) (width 0.05))
+    (fp_line (start 0.25 -0.475) (end -0.25 -0.475) (layer F.SilkS) (width 0.15))
+    (fp_line (start -0.25 0.475) (end 0.25 0.475) (layer F.SilkS) (width 0.15))
+    (pad 1 smd rect (at -0.55 0) (size 0.6 0.5) (layers F.Cu F.Paste F.Mask)
+      (net 1 GND))
+    (pad 2 smd rect (at 0.55 0) (size 0.6 0.5) (layers F.Cu F.Paste F.Mask)
+      (net 3 /VBUS))
+    (model Capacitors_SMD/C_0402.wrl
+      (at (xyz 0 0 0))
+      (scale (xyz 1 1 1))
+      (rotate (xyz 0 0 0))
+    )
+  )
 )

Commit message: Signed-off-by: Chris Stook <chris@chrisstook.com>
Parts:
- added M1: 9575, Keystone_Electronics_Footprints:9575, F.Cu at (142.0, 121.7)
- added M2: 9575, Keystone_Electronics_Footprints:9575, F.Cu at (142.0, 96.7)
- J1: value 10118194-0001LF -> 10118193-0001LF; footprint FCI_Footprints:10118194-0001LF -> FCI_Footprints:10118193-0001LF
- moved D1 57.8 mm to (152.3, 109.2)
- moved J2 47.9 mm to (176.9, 109.0)
- moved J1 43.9 mm to (128.5, 109.2)
- moved U2 0.20 mm to (151.9, 63.0)
Other:
- board outline added: 54.6 x 33 mm
Changed lines of the file:
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@@
 (kicad_pcb (version 4) (host pcbnew 4.0.1-stable)
   (general
-    (links 96)
+    (links 94)
     (no_connects 94)
     (area 0 0 0 0)
     (thickness 1.6)
-    (drawings 0)
+    (drawings 12)
     (tracks 0)
     (zones 0)
-    (modules 35)
-    (nets 44)
+    (modules 37)
+    (nets 46)
   )
   (page A4)
@@
   (net 42 "Net-(U2-Pad13)")
   (net 43 "Net-(U3-Pad1)")
+  (net 44 "Net-(M1-Pad1)")
+  (net 45 "Net-(M2-Pad1)")
   (net_class Default "This is the default net class."
     (clearance 0.2032)
@@
     (add_net "Net-(D1-Pad4)")
     (add_net "Net-(J1-Pad4)")
+    (add_net "Net-(M1-Pad1)")
+    (add_net "Net-(M2-Pad1)")
     (add_net "Net-(R4-Pad2)")
     (add_net "Net-(R5-Pad2)")
@@
   )
   (module Dialight_Footprints:PLCC-4_515-114 (layer F.Cu)
-    (at 141.9225 52.3875 270)
+    (at 152.3238 109.22 270)
     (descr C:\Users\Chris\VendorData\dialight\C17211.pdf)
-    (fp_text reference D1 (at 0 6.6 270) (layer F.SilkS)
+    (fp_text reference D1 (at 2.54 -1.7272 360) (layer F.SilkS)
       (effects (font (size 1 1) (thickness 0.15)))
     )
@@
     (pad "" np_thru_hole circle (at -3.5814 1.6002 270) (size 1.9304 1.9304) (drill 1.9304) (layers *.Cu *.Mask F.SilkS))
   )
-  (module FCI_Footprints:10118194-0001LF (layer F.Cu)
-    (at 125.73 65.405 270)
-    (fp_text reference J1 (at 7 -2 270) (layer F.SilkS)
-      (effects (font (size 1 1) (thickness 0.15)))
-    )
-    (fp_text value 10118194-0001LF (at 0 3 270) (layer F.Fab)
-      (effects (font (size 1 1) (thickness 0.15)))
-    )
-    (fp_line (start 4 -3) (end 3.2 -3) (layer F.SilkS) (width 0.15))
-    (fp_line (start -4 -3) (end -3.2 -3) (layer F.SilkS) (width 0.15))
-    (fp_line (start 4 -1) (end 4 -3) (layer F.SilkS) (width 0.15))
-    (fp_line (start -4 -1) (end -4 -3) (layer F.SilkS) (width 0.15))
-    (fp_line (start -4 1.45) (end 4 1.45) (layer F.SilkS) (width 0.15))
-    (pad 9 smd rect (at -1 0 270) (size 1.5 1.55) (layers F.Cu F.Paste F.Mask)
-      (net 1 GND))
-    (pad 10 smd rect (at 1 0 270) (size 1.5 1.55) (layers F.Cu F.Paste F.Mask)
-      (net 1 GND))
-    (pad 11 smd rect (at 3.05 0 270) (size 1.5 1.55) (layers F.Cu F.Paste F.Mask)
-      (net 1 GND))
-    (pad 8 smd rect (at -3.05 0 270) (size 1.5 1.55) (layers F.Cu F.Paste F.Mask)
-      (net 1 GND))
-    (pad 8 thru_hole circle (at -3.6 0 270) (size 1.55 1.55) (drill 1.15) (layers *.Cu *.Mask F.SilkS)
-      (net 1 GND))
-    (pad 11 thru_hole circle (at 3.6 0 270) (size 1.55 1.55) (drill 1.15) (layers *.Cu *.Mask F.SilkS)
-      (net 1 GND))
-    (pad 3 smd rect (at 0 -2.7 270) (size 0.4 1.35) (layers F.Cu F.Paste F.Mask)
-      (net 12 "Net-(CR1-Pad1)"))
-    (pad 4 smd rect (at 0.65 -2.7 270) (size 0.4 1.35) (layers F.Cu F.Paste F.Mask)
-      (net 18 "Net-(J1-Pad4)"))
-    (pad 5 smd rect (at 1.3 -2.7 270) (size 0.4 1.35) (layers F.Cu F.Paste F.Mask)
-      (net 1 GND))
-    (pad 2 smd rect (at -0.65 -2.7 270) (size 0.4 1.35) (layers F.Cu F.Paste F.Mask)
-      (net 13 "Net-(CR2-Pad1)"))
-    (pad 1 smd rect (at -1.3 -2.7 270) (size 0.4 1.35) (layers F.Cu F.Paste F.Mask)
-      (net 2 "Net-(C1-Pad2)"))
-    (pad 6 thru_hole circle (at -2.5 -2.7 270) (size 1.25 1.25) (drill 0.85) (layers *.Cu *.Mask F.SilkS)
-      (net 1 GND))
-    (pad 7 thru_hole circle (at 2.5 -2.7 270) (size 1.25 1.25) (drill 0.85) (layers *.Cu *.Mask F.SilkS)
-      (net 1 GND))
-  )
   (module Standard_Footprints:C0402 (layer F.Cu)
     (at 130.175 62.23 270)
@@
   )
   (module FTDI_Footprints:LQFP_48 (layer F.Cu)
-    (at 151.765 62.865 180)
+    (at 151.9428 62.9666 180)
     (fp_text reference U2 (at 0 -6.15 180) (layer F.SilkS)
       (effects (font (size 1.2 1.2) (thickness 0.15)))
@@
   )
   (module TE_Connectivity_Footprints:826947-4 (layer F.Cu)
-    (at 166.37 62.23 90)
-    (fp_text reference J2 (at -2.62 -2.5 90) (layer F.SilkS)
+    (at 176.911 108.966 90)
+    (fp_text reference J2 (at -5.969 2.667 180) (layer F.SilkS)
       (effects (font (size 1 1) (thickness 0.15)))
     )
@@
     )
   )
+  (module Keystone_Electronics_Footprints:9575 (layer F.Cu)
+    (at 142.0114 121.6914)
+    (fp_text reference M1 (at -5.1054 -0.0254) (layer F.SilkS)
+      (effects (font (size 1 1) (thickness 0.15)))
+    )
+    (fp_text value 9575 (at -0.1 5.6) (layer F.Fab)
+      (effects (font (size 1 1) (thickness 0.15)))
+    )
+    (pad 1 thru_hole circle (at 0 0) (size 6.2 6.2) (drill 2.8) (layers *.Cu *.Mask F.SilkS)
+      (net 44 "Net-(M1-Pad1)"))
+  )
+  (module Keystone_Electronics_Footprints:9575 (layer F.Cu)
+    (at 142.0114 96.7486)
+    (fp_text reference M2 (at -5.2324 -0.1016) (layer F.SilkS)
+      (effects (font (size 1 1) (thickness 0.15)))
+    )
+    (fp_text value 9575 (at -0.1 5.6) (layer F.Fab)
+      (effects (font (size 1 1) (thickness 0.15)))
+    )
+    (pad 1 thru_hole circle (at 0 0) (size 6.2 6.2) (drill 2.8) (layers *.Cu *.Mask F.SilkS)
+      (net 45 "Net-(M2-Pad1)"))
+  )
+  (module FCI_Footprints:10118193-0001LF (layer F.Cu)
+    (at 128.4732 109.22 270)
+    (fp_text reference J1 (at 5.461 -3.6068 360) (layer F.SilkS)
+      (effects (font (size 1 1) (thickness 0.15)))
+    )
+    (fp_text value 10118193-0001LF (at 0 4.3 270) (layer F.Fab)
+      (effects (font (size 1 1) (thickness 0.15)))
+    )
+    (fp_line (start 4.2 -2.2) (end 4.2 -3.6) (layer F.SilkS) (width 0.15))
+    (fp_line (start 4.2 -3.6) (end 2.6 -3.6) (layer F.SilkS) (width 0.15))
+    (fp_line (start -4.2 -2.2) (end -4.2 -3.6) (layer F.SilkS) (width 0.15))
+    (fp_line (start -4.2 -3.6) (end -2.6 -3.6) (layer F.SilkS) (width 0.15))
+    (fp_line (start -4 1.45) (end 4 1.45) (layer F.SilkS) (width 0.15))
+    (pad 9 smd rect (at -1.2 0 270) (size 1.9 1.6) (layers F.Cu F.Paste F.Mask)
+      (net 1 GND))
+    (pad 10 smd rect (at 1.2 0 270) (size 1.9 1.6) (layers F.Cu F.Paste F.Mask)
+      (net 1 GND))
+    (pad 8 thru_hole circle (at -3.3 0 270) (size 1.6 1.6) (drill 1.2) (layers *.Cu *.Mask F.SilkS)
+      (net 1 GND))
+    (pad 11 thru_hole circle (at 3.3 0 270) (size 1.6 1.6) (drill 1.2) (layers *.Cu *.Mask F.SilkS)
+      (net 1 GND))
+    (pad 3 smd rect (at 0 -2.675 270) (size 0.4 1.35) (layers F.Cu F.Paste F.Mask)
+      (net 12 "Net-(CR1-Pad1)"))
+    (pad 4 smd rect (at 0.65 -2.675 270) (size 0.4 1.35) (layers F.Cu F.Paste F.Mask)
+      (net 18 "Net-(J1-Pad4)"))
+    (pad 5 smd rect (at 1.3 -2.675 270) (size 0.4 1.35) (layers F.Cu F.Paste F.Mask)
+      (net 1 GND))
+    (pad 2 smd rect (at -0.65 -2.675 270) (size 0.4 1.35) (layers F.Cu F.Paste F.Mask)
+      (net 13 "Net-(CR2-Pad1)"))
+    (pad 1 smd rect (at -1.3 -2.675 270) (size 0.4 1.35) (layers F.Cu F.Paste F.Mask)
+      (net 2 "Net-(C1-Pad2)"))
+    (pad 6 smd rect (at -3.2 -2.675 270) (size 1.6 1.4) (layers F.Cu F.Paste F.Mask)
+      (net 1 GND))
+    (pad 7 smd rect (at 3.2 -2.675 270) (size 1.6 1.4) (layers F.Cu F.Paste F.Mask)
+      (net 1 GND))
+  )
+  (gr_line (start 146.05 100.33) (end 146.05 92.71) (angle 90) (layer F.SilkS) (width 0.2))
+  (gr_line (start 130.81 100.33) (end 146.05 100.33) (angle 90) (layer F.SilkS) (width 0.2))
+  (gr_line (start 146.05 118.11) (end 146.05 125.73) (angle 90) (layer F.SilkS) (width 0.2))
+  (gr_line (start 130.81 118.11) (end 146.05 118.11) (angle 90) (layer F.SilkS) (width 0.2))
+  (gr_line (start 127.0254 114.3) (end 130.81 114.3) (angle 90) (layer Edge.Cuts) (width 0.15))
+  (gr_line (start 127.0254 104.14) (end 127.0254 114.3) (angle 90) (layer Edge.Cuts) (width 0.15))
+  (gr_line (start 130.81 104.14) (end 127.0254 104.14) (angle 90) (layer Edge.Cuts) (width 0.15))
+  (gr_line (start 181.61 92.71) (end 130.81 92.71) (angle 90) (layer Edge.Cuts) (width 0.15))
+  (gr_line (start 181.61 125.73) (end 181.61 92.71) (angle 90) (layer Edge.Cuts) (width 0.15))
+  (gr_line (start 130.81 125.73) (end 181.61 125.73) (angle 90) (layer Edge.Cuts) (width 0.15))
+  (gr_line (start 130.81 114.3) (end 130.81 125.73) (angle 90) (layer Edge.Cuts) (width 0.15))
+  (gr_line (start 130.81 92.71) (end 130.81 104.14) (angle 90) (layer Edge.Cuts) (width 0.15))
 )

Commit message: Signed-off-by: Chris Stook <chris@chrisstook.com>
Parts:
- moved R9 73.9 mm to (148.0, 123.1), turned to 0 degrees
- moved C14 72.0 mm to (153.3, 124.5)
- moved R8 68.5 mm to (148.0, 120.9), turned to 0 degrees
- moved U3 66.8 mm to (153.7, 121.8)
- moved C12 60.2 mm to (137.0, 114.8)
- moved R7 58.2 mm to (136.1, 117.0), turned to 0 degrees
- moved R3 55.9 mm to (147.6, 118.7)
- moved C13 55.4 mm to (136.5, 113.0), turned to 0 degrees
- moved CR1 50.3 mm to (134.1, 112.5), turned to 270 degrees
- moved C3 50.1 mm to (149.7, 116.3), turned to 90 degrees
- moved U2 50.0 mm to (143.1, 112.1), turned to 0 degrees
- moved R6 49.4 mm to (151.8, 116.3)
- moved C10 48.9 mm to (137.2, 109.0), turned to 90 degrees
- moved L2 46.2 mm to (142.6, 103.0), turned to 0 degrees
- moved R5 44.4 mm to (134.7, 109.7)
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Routing:
- net /VBUS: track 0.00 -> 30.9 mm
- net /VCCD: track 0.00 -> 28.9 mm
- net Net-(D1-Pad4): track 0.00 -> 28.0 mm
- net Net-(U2-Pad13): track 0.00 -> 19.2 mm
- net Net-(D1-Pad2): track 0.00 -> 17.5 mm
- net /UART_TX: track 0.00 -> 15.7 mm
- net Net-(C3-Pad2): track 0.00 -> 12.9 mm
- net /VBUSDTCT: track 0.00 -> 12.6 mm
- net Net-(C5-Pad2): track 0.00 -> 10.9 mm
- net Net-(C11-Pad2): track 0.00 -> 10.2 mm
- net Net-(C1-Pad2): track 0.00 -> 9.32 mm
- net Net-(R7-Pad2): track 0.00 -> 8.77 mm
- net Net-(D1-Pad3): track 0.00 -> 7.36 mm
- net Net-(R4-Pad2): track 0.00 -> 6.29 mm
- net GND: track 0.00 -> 5.38 mm
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
Commit message: Signed-off-by: Chris Stook <chris@chrisstook.com>
Parts:
- moved R1 1.45 mm to (152.3, 97.9)
- moved R2 1.45 mm to (149.4, 94.5)
- moved U1 1.45 mm to (149.4, 97.9)
- moved C10 0.18 mm to (137.0, 108.8)
Routing:
- net GND: track 5.38 -> 78.8 mm, vias 0 -> 30
- net /VBUS: track 30.9 -> 90.2 mm, vias 0 -> 3
- net /VCCD: track 28.9 -> 83.3 mm, vias 0 -> 6
- net /UART_RX: track 0.00 -> 47.2 mm, vias 0 -> 1
- net /VPHY: track 2.43 -> 22.8 mm, vias 0 -> 2
- net /EE_CS: track 0.00 -> 19.9 mm, vias 0 -> 2
- net /EE_DATA: track 2.21 -> 21.9 mm
- net /EE_CLK: track 0.00 -> 17.6 mm, vias 0 -> 2
- net /VPLL: track 1.90 -> 18.9 mm, vias 0 -> 4
- net /VBUSDTCT: track 12.6 -> 16.0 mm, vias 0 -> 2
- net Net-(R7-Pad2): track 8.77 -> 11.8 mm
- net Net-(C3-Pad2): track 12.9 -> 11.5 mm
- net Net-(U2-Pad13): track 19.2 -> 20.2 mm
- added copper zone on B.Cu, net GND
Other:
- board size 54.6 x 33 mm -> 35.5 x 33 mm

Commit message: Signed-off-by: Chris Stook <chris@chrisstook.com>
Parts:
- added C15: C1005X7R1H104K050BB, Standard_Footprints:C0402, F.Cu at (152.4, 100.1)
- added J3: 5019, Keystone_Electronics_Footprints:5090, F.Cu at (157.5, 96.0)
- C11, C5: value 04025A100JAT2A -> 04025A180JAT2A
- X1: value ABM10AIG-12.000MHZ-4Z-T3 -> ABM8G-12.000MHZ-18-D2Y-T; footprint Abracon_Footprints:ABM10AIG -> Abracon_Footprints:ABM8G
- moved X1 0.48 mm to (137.4, 102.5)
- moved C11 0.38 mm to (134.7, 102.1)
- moved L1 0.25 mm to (133.5, 102.1)
Routing:
- net GND: track 78.8 -> 86.1 mm, vias 30 -> 32
- net /EE_CLK: track 17.6 -> 18.4 mm
- net /VPHY: track 22.8 -> 23.5 mm
- added copper zone on F.Cu, net /VCCD
