File: kicad/PSP-603_USB.kicad_pcb (KiCad board)
At the start: 2 copper layers, 34 x 33 mm, 17 parts, among them J1 10118193-0001LF, J2 5019, J3 826947-4, M1 9575, M2 9575, U1 FT232RL-REEL

Commit message: Signed-off-by: Chris Stook <chris@chrisstook.com>
Other:
- board text added: "PSP-603 USB 4/23/2016"
- board text removed: "PSP-603 USB 3/26/2016"
Changed lines of the file:
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@@
   (general
     (links 42)
-    (no_connects 1)
-    (area 128.450399 92.634999 162.635001 125.805001)
+    (no_connects 0)
+    (area 124.4942 92.609999 162.635001 129.5454)
     (thickness 1.6)
     (drawings 15)
@@
     (effects (font (size 1.5 1.5) (thickness 0.3)) (justify left))
   )
-  (gr_text "PSP-603 USB\n3/26/2016" (at 153.4 118.6) (layer B.SilkS)
+  (gr_text "PSP-603 USB\n4/23/2016" (at 153.4 118.6) (layer B.SilkS)
     (effects (font (size 1.5 1.5) (thickness 0.3)) (justify mirror))
   )
