File: kicad/PSP-603_USB.sch (KiCad schematic (older format))
At the start: 33 parts, among them J1 10118194-0001LF, J2 826947-4, U1 93LC56BT-I/OT, U2 FT232HL-Reel, X1 ABM10AIG-12.000MHZ-4Z-T3

Commit message: Signed-off-by: Chris Stook <chris@chrisstook.com>
Parts:
- added C14: C1005X7R1H104K050BB, Standard_Footprints:C0402, symbol C1005X7R1H104K050BB
- added U3: SN74LV1T34DBVR, Standard_Footprints:TSOT-23-5, symbol SN74LV1T34DBVR
Connections:
- wire segments 147 -> 158
- no-connect marks 14 -> 15
Other:
- moved on the sheet: J2
Changed lines of the file:
@@
 LIBS:AVX_Library
 LIBS:TE_Connectivity_Library
+LIBS:TI_Library
 LIBS:PSP-603_USB-cache
 EELAYER 25 0
@@
 	6550 5850 6600 5850
 Wire Wire Line
-	6550 6200 6850 6200
-Wire Wire Line
-	6850 6200 6850 5650
+	6850 6200 6550 6200
+Wire Wire Line
+	6850 5650 6850 6200
 Wire Wire Line
 	6850 5650 6200 5650
@@
 	2500 5250 2500 4950
 Wire Wire Line
-	8350 2900 9850 2900
-Wire Wire Line
-	8350 3000 9850 3000
-Text Label 9350 2900 0    60   ~ 0
+	8350 3000 10100 3000
+Text Label 9700 2900 0    60   ~ 0
 UART_TX
-Text Label 9350 3000 0    60   ~ 0
+Text Label 9700 3000 0    60   ~ 0
 UART_RX
 $Comp
@@
 	9350 3150 9350 3100
 Wire Wire Line
-	9350 3100 9850 3100
-Wire Wire Line
-	2100 1150 9150 1150
-Wire Wire Line
-	9150 1150 9150 2800
-Wire Wire Line
-	9150 2800 9850 2800
+	9350 3100 10100 3100
+Wire Wire Line
+	2100 1150 9750 1150
+Wire Wire Line
+	9750 1150 9750 2800
+Wire Wire Line
+	9750 2800 10100 2800
 Connection ~ 2100 2050
-Text Label 9350 2800 0    60   ~ 0
+Text Label 9800 2800 0    60   ~ 0
 VBUS
 Connection ~ 2500 4950
@@
 L 826947-4 J2
 U 1 1 56C9F91B
-P 9950 2950
-F 0 "J2" H 10000 2700 60  0000 C CNN
-F 1 "826947-4" H 10000 2600 60  0000 C CNN
-F 2 "TE_Connectivity_Footprints:826947-4" H 10000 1600 60  0001 C CNN
-F 3 "C:/Users/Chris/VendorData/TE Connectivity/ENG_CD_826629_AA_baseFilename.pdf" H 9950 1500 60  0001 C CNN
-F 4 "TE Connectivity" H 10050 2400 60  0001 C CNN "mfg"
-F 5 "826947-4" H 10000 2300 60  0001 C CNN "mfg part number"
-F 6 "0.1\"" H 10000 2200 60  0001 C CNN "Pitch"
-F 7 "0.264\"" H 10000 2100 60  0001 C CNN "Contact Mating Length"
-F 8 "Solder" H 10000 2000 60  0001 C CNN "Termination"
-F 9 "tin" H 10000 1900 60  0001 C CNN "Finish"
-F 10 "green" H 10000 1800 60  0001 C CNN "Color"
-F 11 "Square" H 10000 1700 60  0001 C CNN "Pin Shape"
-	1    9950 2950
-	1    0    0    -1
-$EndComp
+P 10200 2950
+F 0 "J2" H 10250 2700 60  0000 C CNN
+F 1 "826947-4" H 10250 2600 60  0000 C CNN
+F 2 "TE_Connectivity_Footprints:826947-4" H 10250 1600 60  0001 C CNN
+F 3 "C:/Users/Chris/VendorData/TE Connectivity/ENG_CD_826629_AA_baseFilename.pdf" H 10200 1500 60  0001 C CNN
+F 4 "TE Connectivity" H 10300 2400 60  0001 C CNN "mfg"
+F 5 "826947-4" H 10250 2300 60  0001 C CNN "mfg part number"
+F 6 "0.1\"" H 10250 2200 60  0001 C CNN "Pitch"
+F 7 "0.264\"" H 10250 2100 60  0001 C CNN "Contact Mating Length"
+F 8 "Solder" H 10250 2000 60  0001 C CNN "Termination"
+F 9 "tin" H 10250 1900 60  0001 C CNN "Finish"
+F 10 "green" H 10250 1800 60  0001 C CNN "Color"
+F 11 "Square" H 10250 1700 60  0001 C CNN "Pin Shape"
+	1    10200 2950
+	1    0    0    -1
+$EndComp
+$Comp
+L SN74LV1T34DBVR U3
+U 1 1 56C8E4E0
+P 9300 2800
+F 0 "U3" H 9400 2900 60  0000 C CNN
+F 1 "SN74LV1T34DBVR" H 9300 3000 60  0000 C CNN
+F 2 "Standard_Footprints:TSOT-23-5" H 9300 2050 60  0001 C CNN
+F 3 "C:/Users/Chris/VendorData/TI/sn74lv1t34.pdf" H 9300 2150 60  0001 C CNN
+F 4 "TI" H 9250 2350 60  0001 C CNN "mfg"
+F 5 "SN74LV1T34DBVR" H 9250 2250 60  0001 C CNN "mfg part number"
+	1    9300 2800
+	1    0    0    -1
+$EndComp
+$Comp
+L GND #PWR025
+U 1 1 56C8EB31
+P 3400 7600
+F 0 "#PWR025" H 3400 7350 50  0001 C CNN
+F 1 "GND" H 3400 7450 50  0000 C CNN
+F 2 "" H 3400 7600 50  0000 C CNN
+F 3 "" H 3400 7600 50  0000 C CNN
+	1    3400 7600
+	1    0    0    -1
+$EndComp
+$Comp
+L SN74LV1T34DBVR U3
+U 2 1 56C8EFB3
+P 3400 7150
+F 0 "U3" H 3650 7050 60  0000 C CNN
+F 1 "SN74LV1T34DBVR" H 3950 6950 60  0000 C CNN
+F 2 "Standard_Footprints:TSOT-23-5" H 3400 6400 60  0001 C CNN
+F 3 "C:/Users/Chris/VendorData/TI/sn74lv1t34.pdf" H 3400 6500 60  0001 C CNN
+F 4 "TI" H 3350 6700 60  0001 C CNN "mfg"
+F 5 "SN74LV1T34DBVR" H 3350 6600 60  0001 C CNN "mfg part number"
+	2    3400 7150
+	1    0    0    -1
+$EndComp
+Wire Wire Line
+	3400 7600 3400 7500
+Wire Wire Line
+	3400 6800 3400 6700
+Wire Wire Line
+	2950 6700 3650 6700
+Text Label 3400 6700 0    60   ~ 0
+VBUS
+NoConn ~ 3200 7150
+Wire Wire Line
+	8350 2900 9000 2900
+Wire Wire Line
+	9000 2900 9000 2800
+Wire Wire Line
+	9000 2800 9100 2800
+Wire Wire Line
+	9500 2800 9600 2800
+Wire Wire Line
+	9600 2800 9600 2900
+Wire Wire Line
+	9600 2900 10100 2900
+$Comp
+L C1005X7R1H104K050BB C14
+U 1 1 56C91386
+P 2950 7150
+F 0 "C14" V 2750 6950 60  0000 C CNN
+F 1 "C1005X7R1H104K050BB" H 3050 6600 60  0001 C CNN
+F 2 "Standard_Footprints:C0402" H 3000 6900 60  0001 C CNN
+F 3 "" H 2950 7000 60  0000 C CNN
+F 4 "TDK" H 3000 6800 60  0001 C CNN "mfg"
+F 5 "C1005X7R1H104K050BB" H 3050 6700 60  0001 C CNN "mfg part number"
+F 6 "0.1uF" V 2850 7000 60  0000 C CNN "Capacatance"
+F 7 "50V" H 2950 6500 60  0001 C CNN "Voltage"
+F 8 "+/- 10%" H 2950 6400 60  0001 C CNN "Tolerance"
+F 9 "X7R" H 2950 6300 60  0001 C CNN "Dielectric"
+F 10 "-55C / +125C" H 2950 6200 60  0001 C CNN "Temp Range"
+	1    2950 7150
+	0    1    1    0
+$EndComp
+Wire Wire Line
+	2950 6700 2950 7000
+Connection ~ 3400 6700
+Wire Wire Line
+	3400 7550 2950 7550
+Wire Wire Line
+	2950 7550 2950 7300
+Connection ~ 3400 7550
 $EndSCHEMATC

Commit message: Signed-off-by: Chris Stook <chris@chrisstook.com>
Parts:
- removed J1: 10118194-0001LF, FCI_Footprints:10118194-0001LF, symbol 10118194-0001LF
- added J1: 10118193-0001LF, FCI_Footprints:10118193-0001LF, symbol 10118193-0001LF
- added M1, M2: 9575, Keystone_Electronics_Footprints:9575, symbol 9575
Connections:
- no-connect marks 15 -> 17
Changed lines of the file:
@@
 LIBS:power
 LIBS:FCI_Library
-LIBS:FTDI
 LIBS:Abracon_Library
 LIBS:Microchip_Library
@@
 LIBS:TE_Connectivity_Library
 LIBS:TI_Library
+LIBS:FTDI_Library
+LIBS:Keystone_Electronics_Library
 LIBS:PSP-603_USB-cache
 EELAYER 25 0
@@
 	1    6250 6050
 	0    -1   -1   0
-$EndComp
-$Comp
-L 10118194-0001LF J1
-U 1 1 56C7A421
-P 1250 3600
-F 0 "J1" H 1150 3900 60  0000 C CNN
-F 1 "10118194-0001LF" H 1500 4000 60  0000 C CNN
-F 2 "FCI_Footprints:10118194-0001LF" H 1400 2850 60  0001 C CNN
-F 3 "C:/Users/Chris/VendorData/FCI/10118194.pdf" H 1400 2950 60  0001 C CNN
-F 4 "FCI" H 1300 3150 60  0001 C CNN "mfg"
-F 5 "10118194-0001LF" H 1300 3050 60  0001 C CNN "mfg part number"
-	1    1250 3600
-	1    0    0    -1
 $EndComp
 $Comp
@@
 	2950 7550 2950 7300
 Connection ~ 3400 7550
+$Comp
+L 9575 M1
+U 1 1 56CE57F1
+P 4750 7100
+F 0 "M1" V 4900 7100 60  0000 C CNN
+F 1 "9575" V 5000 7100 60  0000 C CNN
+F 2 "Keystone_Electronics_Footprints:9575" H 4800 6450 60  0001 C CNN
+F 3 "C:/Users/Chris/VendorData/Keystone Electronics/9575-9581 (self tapping screw).PDF" H 5350 6550 60  0001 C CNN
+F 4 "Keystone Electronics" H 4800 6750 60  0001 C CNN "mfg"
+F 5 "9575" H 4750 6650 60  0001 C CNN "mfg part number"
+	1    4750 7100
+	0    -1   -1   0
+$EndComp
+$Comp
+L 9575 M2
+U 1 1 56CE5C33
+P 5050 7100
+F 0 "M2" V 5200 7100 60  0000 C CNN
+F 1 "9575" V 5300 7100 60  0000 C CNN
+F 2 "Keystone_Electronics_Footprints:9575" H 5100 6450 60  0001 C CNN
+F 3 "C:/Users/Chris/VendorData/Keystone Electronics/9575-9581 (self tapping screw).PDF" H 5650 6550 60  0001 C CNN
+F 4 "Keystone Electronics" H 5100 6750 60  0001 C CNN "mfg"
+F 5 "9575" H 5050 6650 60  0001 C CNN "mfg part number"
+	1    5050 7100
+	0    -1   -1   0
+$EndComp
+NoConn ~ 4750 7250
+NoConn ~ 5050 7250
+$Comp
+L 10118193-0001LF J1
+U 1 1 56CE96CD
+P 1250 3600
+F 0 "J1" H 1150 3900 60  0000 C CNN
+F 1 "10118193-0001LF" H 1500 4000 60  0000 C CNN
+F 2 "FCI_Footprints:10118193-0001LF" H 1400 2850 60  0001 C CNN
+F 3 "C:/Users/Chris/VendorData/FCI/10118193.pdf" H 1400 2950 60  0001 C CNN
+F 4 "FCI" H 1300 3150 60  0001 C CNN "mfg"
+F 5 "10118193-0001LF" H 1300 3050 60  0001 C CNN "mfg part number"
+	1    1250 3600
+	1    0    0    -1
+$EndComp
 $EndSCHEMATC

Commit message: Signed-off-by: Chris Stook <chris@chrisstook.com>
Parts:
- removed C11, C5: 04025A100JAT2A, Standard_Footprints:C0402, symbol 04025A100JAT2A
- removed X1: ABM10AIG-12.000MHZ-4Z-T3, Abracon_Footprints:ABM10AIG, symbol ABM10AIG-12.000MHZ-4Z-T3
- added C11, C5: 04025A180JAT2A, Standard_Footprints:C0402, symbol 04025A180JAT2A
- added C15: C1005X7R1H104K050BB, Standard_Footprints:C0402, symbol C1005X7R1H104K050BB
- added J3: 5019, Keystone_Electronics_Footprints:5090, symbol 5019
- added X1: ABM8G-12.000MHZ-18-D2Y-T, Abracon_Footprints:ABM8G, symbol ABM8G-12.000MHZ-18-D2Y-T
Connections:
- wire segments 158 -> 162
Changed lines of the file:
@@
 $EndDescr
-$Comp
-L ABM10AIG-12.000MHZ-4Z-T3 X1
-U 1 1 56C7A3C3
-P 6250 6050
-F 0 "X1" V 5950 6150 60  0000 C CNN
-F 1 "ABM10AIG-12.000MHZ-4Z-T3" H 7200 5350 60  0001 C CNN
-F 2 "Abracon_Footprints:ABM10AIG" H 7150 5450 60  0001 C CNN
-F 3 "C:/Users/Chris/VendorData/Abracon/ABM10AIG.pdf" H 7700 5250 60  0001 C CNN
-F 4 "Abracon" H 6700 6250 60  0001 C CNN "mfg"
-F 5 "ABM10AIG-12.000MHZ-4Z-T3" H 7200 5950 60  0001 C CNN "mfg number"
-F 6 "10pF" H 6650 5850 60  0001 C CNN "Load Capacatance"
-F 7 "150 Ohm" H 6750 5750 60  0001 C CNN "ESR"
-F 8 "+/- 50ppm" H 6800 5650 60  0001 C CNN "Frequency Stability"
-F 9 "+/- 30ppm" H 6800 5550 60  0001 C CNN "Frequency Tolerance"
-F 10 "12MHz" V 5850 6050 60  0000 C CNN "Frequency"
-	1    6250 6050
-	0    -1   -1   0
-$EndComp
 $Comp
 L FT232HL-Reel U2
@@
 	1600 5350 1600 5450
 Wire Wire Line
-	2400 5250 2500 5250
-Wire Wire Line
-	2450 4950 2950 4950
+	2500 5250 2400 5250
+Wire Wire Line
+	2450 4950 2500 4950
+Wire Wire Line
+	2500 4650 2500 5250
 Wire Wire Line
 	1450 5250 1800 5250
@@
 	1    0    0    -1
 $EndComp
-Wire Wire Line
-	2500 5250 2500 4950
 Wire Wire Line
 	8350 3000 10100 3000
@@
 VBUS
 Connection ~ 2500 4950
-Text Label 2850 4950 2    60   ~ 0
+Text Label 3200 4650 2    60   ~ 0
 VCCD
 NoConn ~ 1550 3700
@@
 Text Label 7200 1500 2    60   ~ 0
 VCCD
-$Comp
-L 04025A100JAT2A C5
-U 1 1 56C9AE48
-P 5550 6050
-F 0 "C5" V 5500 5750 60  0000 C CNN
-F 1 "04025A100JAT2A" H 5650 5500 60  0001 C CNN
-F 2 "Standard_Footprints:C0402" H 5600 5800 60  0001 C CNN
-F 3 "C:/Users/Chris/VendorData/AVX/C0GNP0-Dielectric.pdf" H 5600 5000 60  0001 C CNN
-F 4 "AVX" H 5600 5700 60  0001 C CNN "mfg"
-F 5 "04025A100JAT2A" H 5650 5600 60  0001 C CNN "mfg part number"
-F 6 "10pF" V 5600 5800 60  0000 C CNN "Capacatance"
-F 7 "50V" H 5550 5400 60  0001 C CNN "Voltage"
-F 8 "+/- 5%" H 5550 5300 60  0001 C CNN "Tolerance"
-F 9 "NPO" H 5550 5200 60  0001 C CNN "Dielectric"
-F 10 "-55C / +125C" H 5550 5100 60  0001 C CNN "Temp Range"
-	1    5550 6050
-	0    1    1    0
-$EndComp
 Wire Wire Line
 	2450 5950 2600 5950
@@
 Wire Wire Line
 	5550 5850 6000 5850
-$Comp
-L 04025A100JAT2A C11
-U 1 1 56C9CBD1
-P 7050 6050
-F 0 "C11" V 7000 5750 60  0000 C CNN
-F 1 "04025A100JAT2A" H 7150 5500 60  0001 C CNN
-F 2 "Standard_Footprints:C0402" H 7100 5800 60  0001 C CNN
-F 3 "C:/Users/Chris/VendorData/AVX/C0GNP0-Dielectric.pdf" H 7100 5000 60  0001 C CNN
-F 4 "AVX" H 7100 5700 60  0001 C CNN "mfg"
-F 5 "04025A100JAT2A" H 7150 5600 60  0001 C CNN "mfg part number"
-F 6 "10pF" V 7100 5800 60  0000 C CNN "Capacatance"
-F 7 "50V" H 7050 5400 60  0001 C CNN "Voltage"
-F 8 "+/- 5%" H 7050 5300 60  0001 C CNN "Tolerance"
-F 9 "NPO" H 7050 5200 60  0001 C CNN "Dielectric"
-F 10 "-55C / +125C" H 7050 5100 60  0001 C CNN "Temp Range"
-	1    7050 6050
-	0    -1   1    0
-$EndComp
 $Comp
 L GND #PWR023
@@
 $EndComp
 Wire Wire Line
-	3400 7600 3400 7500
+	3400 7500 3400 7600
 Wire Wire Line
 	3400 6800 3400 6700
@@
 	1    0    0    -1
 $EndComp
+$Comp
+L C1005X7R1H104K050BB C15
+U 1 1 56CFE654
+P 2850 4950
+F 0 "C15" V 2650 4750 60  0000 C CNN
+F 1 "C1005X7R1H104K050BB" H 2950 4400 60  0001 C CNN
+F 2 "Standard_Footprints:C0402" H 2900 4700 60  0001 C CNN
+F 3 "" H 2850 4800 60  0000 C CNN
+F 4 "TDK" H 2900 4600 60  0001 C CNN "mfg"
+F 5 "C1005X7R1H104K050BB" H 2950 4500 60  0001 C CNN "mfg part number"
+F 6 "0.1uF" V 2750 4800 60  0000 C CNN "Capacatance"
+F 7 "50V" H 2850 4300 60  0001 C CNN "Voltage"
+F 8 "+/- 10%" H 2850 4200 60  0001 C CNN "Tolerance"
+F 9 "X7R" H 2850 4100 60  0001 C CNN "Dielectric"
+F 10 "-55C / +125C" H 2850 4000 60  0001 C CNN "Temp Range"
+	1    2850 4950
+	0    1    1    0
+$EndComp
+Wire Wire Line
+	2500 4650 3250 4650
+Wire Wire Line
+	2850 4800 2850 4650
+Connection ~ 2850 4650
+$Comp
+L GND #PWR026
+U 1 1 56CFF306
+P 2850 5150
+F 0 "#PWR026" H 2850 4900 50  0001 C CNN
+F 1 "GND" H 2850 5000 50  0000 C CNN
+F 2 "" H 2850 5150 50  0000 C CNN
+F 3 "" H 2850 5150 50  0000 C CNN
+	1    2850 5150
+	1    0    0    -1
+$EndComp
+Wire Wire Line
+	2850 5100 2850 5150
+$Comp
+L 5019 J3
+U 1 1 56CFFE62
+P 5500 7150
+F 0 "J3" V 5700 7150 60  0000 C CNN
+F 1 "5019" V 5800 7150 60  0000 C CNN
+F 2 "Keystone_Electronics_Footprints:5090" H 5550 6650 60  0001 C CNN
+F 3 "" H 5500 6700 60  0000 C CNN
+F 4 "Keystone Electronics" H 5500 6850 60  0001 C CNN "mfg"
+F 5 "5019" H 5500 6750 60  0001 C CNN "mfg part number"
+	1    5500 7150
+	0    -1   -1   0
+$EndComp
+$Comp
+L GND #PWR027
+U 1 1 56D0041B
+P 5500 7250
+F 0 "#PWR027" H 5500 7000 50  0001 C CNN
+F 1 "GND" H 5500 7100 50  0000 C CNN
+F 2 "" H 5500 7250 50  0000 C CNN
+F 3 "" H 5500 7250 50  0000 C CNN
+	1    5500 7250
+	1    0    0    -1
+$EndComp
+Wire Wire Line
+	5500 7200 5500 7250
+$Comp
+L ABM8G-12.000MHZ-18-D2Y-T X1
+U 1 1 56D01C0D
+P 6250 6050
+F 0 "X1" V 5950 6150 60  0000 C CNN
+F 1 "ABM8G-12.000MHZ-18-D2Y-T" H 7200 5350 60  0001 C CNN
+F 2 "Abracon_Footprints:ABM8G" H 7150 5450 60  0001 C CNN
+F 3 "C:/Users/Chris/VendorData/Abracon/ABM8G.pdf" H 7700 5250 60  0001 C CNN
+F 4 "Abracon" H 6700 6250 60  0001 C CNN "mfg"
+F 5 "ABM8G-12.000MHZ-18-D2Y-T" H 7200 5950 60  0001 C CNN "mfg number"
+F 6 "18pF" H 6650 5850 60  0001 C CNN "Load Capacatance"
+F 7 "150 Ohm" H 6750 5750 60  0001 C CNN "ESR"
+F 8 "+/- 30ppm" H 6800 5650 60  0001 C CNN "Frequency Stability"
+F 9 "+/- 20ppm" H 6800 5550 60  0001 C CNN "Frequency Tolerance"
+F 10 "12MHz" V 5850 6050 60  0000 C CNN "Frequency"
+	1    6250 6050
+	0    -1   -1   0
+$EndComp
+$Comp
+L 04025A180JAT2A C11
+U 1 1 56D0209D
+P 7050 6050
+F 0 "C11" V 6950 6250 60  0000 C CNN
+F 1 "04025A180JAT2A" H 7150 5500 60  0001 C CNN
+F 2 "Standard_Footprints:C0402" H 7100 5800 60  0001 C CNN
+F 3 "C:/Users/Chris/VendorData/AVX/C0GNP0-Dielectric.pdf" H 7100 5000 60  0001 C CNN
+F 4 "AVX" H 7100 5700 60  0001 C CNN "mfg"
+F 5 "04025A180JAT2A" H 7150 5600 60  0001 C CNN "mfg part number"
+F 6 "18pF" V 7050 6300 60  0000 C CNN "Capacatance"
+F 7 "50V" H 7050 5400 60  0001 C CNN "Voltage"
+F 8 "+/- 5%" H 7050 5300 60  0001 C CNN "Tolerance"
+F 9 "NPO" H 7050 5200 60  0001 C CNN "Dielectric"
+F 10 "-55C / +125C" H 7050 5100 60  0001 C CNN "Temp Range"
+	1    7050 6050
+	0    1    1    0
+$EndComp
+$Comp
+L 04025A180JAT2A C5
+U 1 1 56D0257B
+P 5550 6050
+F 0 "C5" V 5450 5750 60  0000 C CNN
+F 1 "04025A180JAT2A" H 5650 5500 60  0001 C CNN
+F 2 "Standard_Footprints:C0402" H 5600 5800 60  0001 C CNN
+F 3 "C:/Users/Chris/VendorData/AVX/C0GNP0-Dielectric.pdf" H 5600 5000 60  0001 C CNN
+F 4 "AVX" H 5600 5700 60  0001 C CNN "mfg"
+F 5 "04025A180JAT2A" H 5650 5600 60  0001 C CNN "mfg part number"
+F 6 "18pF" V 5550 5800 60  0000 C CNN "Capacatance"
+F 7 "50V" H 5550 5400 60  0001 C CNN "Voltage"
+F 8 "+/- 5%" H 5550 5300 60  0001 C CNN "Tolerance"
+F 9 "NPO" H 5550 5200 60  0001 C CNN "Dielectric"
+F 10 "-55C / +125C" H 5550 5100 60  0001 C CNN "Temp Range"
+	1    5550 6050
+	0    1    1    0
+$EndComp
 $EndSCHEMATC
